Commit message: configured simplified camera arm with ros_control support and joystick
necesarry is manual fix of joy_teleop package provided in separated repo

File: description_simple/camera.xacro (robot description, xacro)
@@ -1,22 +1,54 @@
 <?xml version="1.0"?>
 <robot xmlns:xacro="http://www.ros.org/wiki/xacro" >
-    <joint name="camera_joint" type="fixed">
-        <parent link="chassis"/>
+    <xacro:include filename="inertial_macros.xacro"/>
+    <joint name="camera_pan_joint" type="continuous">
+        <parent link="base_link"/>
+        <child link="camera_pan"/>
+        <origin xyz="0.125 0 0.08" rpy="0 0 0"/>
+        <axis xyz="0 0 1"/>
+        <limit effort="1" velocity="20" />
+        <joint_properties friction="4.01"/>
+    </joint>
+    <link name="camera_pan">
+        <visual>
+            <geometry>
+                <box size="0.01 0.01 0.05"/>
+            </geometry>
+            <material name="black"/>
+        </visual>
+        <xacro:inertial_box mass="0.05" x="0.01 " y="0.01" z="0.05">
+            <origin xyz="${0.01/2} 0 ${0.05/2}" rpy="0 0 0"/>
+        </xacro:inertial_box>
+    </link>
+    <joint name="camera_tilt_joint" type="continuous">
+        <parent link="camera_pan"/>
+        <child link="camera_tilt"/>
+        <origin xyz="0.01 0 0.025" rpy="0 0 0"/>
+        <axis xyz="0 1 0"/>
+        <limit effort="1" velocity="20" />
+        <joint_properties friction="4.01"/>
+    </joint>
+    <link name="camera_tilt">
+        <visual>
+            <geometry>
+                <box size="0.01 0.04 0.03"/>
+            </geometry>
+            <material name="black"/>
+        </visual>
+        <xacro:inertial_box mass="0.05" x="0.01 " y="0.05" z="0.05">
+            <origin xyz="${0.01/2} 0 ${0.05/2}" rpy="0 0 0"/>
+        </xacro:inertial_box>
+    </link>
+    <joint name="camera_link_joint" type="fixed">
+        <parent link="camera_tilt"/>
         <child link="camera_link"/>
-        <origin xyz="0.2 0 0.075" rpy="0 0 0"/>
+        <origin xyz="0.01 0 0" rpy="0 0 0"/>
     </joint>
     <link name="camera_link">
         <visual>
             <geometry>
-                <box size="0.010 0.03 0.03"/>
+                <box size="0.01 0.03 0.03"/>
             </geometry>
-            <material name="black"/>
-        </visual>
-        <visual>
-            <origin xyz="0 0 -0.05"/>
-            <geometry>
-                <cylinder radius="0.002" length="0.1"/>
-            </geometry>
-            <material name="black"/>
+            <material name="red"/>
         </visual>
     </link>
@@ -24,5 +56,5 @@
         <parent link="camera_link"/>
         <child link="camera_link_optical"/>
-        <origin xyz="0 0 0" rpy="${-pi/2} 0 ${-pi/2}"/>
+        <origin xyz="0 0 0" rpy="0 0 0"/>
     </joint>
     <link name="camera_link_optical"></link>

File: description_simple/lidar.xacro (robot description, xacro)
@@ -4,5 +4,5 @@
         <parent link="chassis"/>
         <child link="laser_frame"/>
-        <origin xyz="0.135 0 0.095" rpy="0 0 0"/>
+        <origin xyz="0.135 0 0.12" rpy="0 0 0"/>
     </joint>
     <link name="laser_frame">

File: description_simple/ros2_control.xacro (robot description, xacro)
@@ -21,4 +21,26 @@
             <state_interface name="position"/>
         </joint>
+        <joint name="camera_pan_joint">
+            <command_interface name="position">
+                <param name="min">-3.14</param>
+                <param name="max">3.14</param>
+            </command_interface>
+            <state_interface name="position">
+                <param name="initial_value">0</param>
+            </state_interface>
+            <!-- <state_interface name="velocity"/> -->
+            <!-- <state_interface name="effort"/> -->
+        </joint>
+        <joint name="camera_tilt_joint">
+            <command_interface name="position">
+                <param name="min">-3.14</param>
+                <param name="max">3.14</param>
+            </command_interface>
+            <state_interface name="position">
+                <param name="initial_value">0</param>
+            </state_interface>
+            <!-- <state_interface name="velocity"/> -->
+            <!-- <state_interface name="effort"/> -->
+        </joint>
     </ros2_control>
     <gazebo>

Commit message: limited joints for camera

File: description_simple/camera.xacro (robot description, xacro)
@@ -2,11 +2,11 @@
 <robot xmlns:xacro="http://www.ros.org/wiki/xacro" >
     <xacro:include filename="inertial_macros.xacro"/>
-    <joint name="camera_pan_joint" type="continuous">
+    <joint name="camera_pan_joint" type="revolute">
         <parent link="base_link"/>
         <child link="camera_pan"/>
         <origin xyz="0.125 0 0.08" rpy="0 0 0"/>
         <axis xyz="0 0 1"/>
-        <limit effort="1" velocity="20" />
-        <joint_properties friction="4.01"/>
+        <limit effort="1000.0" lower="${-pi/2}" upper="${pi/2}" velocity="2.5"/>
+        <joint_properties friction="1000" damping="10"/>
     </joint>
     <link name="camera_pan">
@@ -21,11 +21,11 @@
         </xacro:inertial_box>
     </link>
-    <joint name="camera_tilt_joint" type="continuous">
+    <joint name="camera_tilt_joint" type="revolute">
         <parent link="camera_pan"/>
         <child link="camera_tilt"/>
         <origin xyz="0.01 0 0.025" rpy="0 0 0"/>
         <axis xyz="0 1 0"/>
-        <limit effort="1" velocity="20" />
-        <joint_properties friction="4.01"/>
+        <limit effort="1000.0" lower="${-pi/2}" upper="${pi/2}" velocity="2.5"/>
+        <joint_properties friction="1000" damping="10"/>
     </joint>
     <link name="camera_tilt">
@@ -36,5 +36,5 @@
             <material name="black"/>
         </visual>
-        <xacro:inertial_box mass="0.05" x="0.01 " y="0.05" z="0.05">
+        <xacro:inertial_box mass="0.01" x="0.01 " y="0.05" z="0.05">
             <origin xyz="${0.01/2} 0 ${0.05/2}" rpy="0 0 0"/>
         </xacro:inertial_box>
