Commit message: moved lidar up to be above the camera

File: description_simple/lidar.xacro (robot description, xacro)
@@ -4,5 +4,5 @@
         <parent link="chassis"/>
         <child link="laser_frame"/>
-        <origin xyz="0.135 0 0.12" rpy="0 0 0"/>
+        <origin xyz="0.135 0 0.15" rpy="0 0 0"/>
     </joint>
     <link name="laser_frame">
@@ -14,7 +14,7 @@
         </visual>
         <visual>
-            <origin xyz="0 0 -0.025"/>
+            <origin xyz="0 0 -0.05"/>
             <geometry>
-                <cylinder radius="0.005" length="0.05"/>
+                <cylinder radius="0.005" length="0.1"/>
             </geometry>
             <material name="black"/>
