Commit message: added params to xacro and launch

File: description_simple/ros2_control.xacro (robot description, xacro)
@@ -1,47 +1,80 @@
 <?xml version="1.0"?>
 <robot xmlns:xacro="http://www.ros.org/wiki/xacro">
-    <ros2_control name="GazeboSystem" type="system">
-        <hardware>
-            <plugin>gazebo_ros2_control/GazeboSystem</plugin>
-        </hardware>
-        <joint name="left_wheel">
-            <command_interface name="velocity">
-                <param name="min">-10</param>
-                <param name="max">10</param>
-            </command_interface>
-            <state_interface name="velocity"/>
-            <state_interface name="position"/>
-        </joint>
-        <joint name="right_wheel">
-            <command_interface name="velocity">
-                <param name="min">-10</param>
-                <param name="max">10</param>
-            </command_interface>
-            <state_interface name="velocity"/>
-            <state_interface name="position"/>
-        </joint>
-        <joint name="camera_pan_joint">
-            <command_interface name="position">
-                <param name="min">-3.14</param>
-                <param name="max">3.14</param>
-            </command_interface>
-            <state_interface name="position">
-                <param name="initial_value">0</param>
-            </state_interface>
-            <!-- <state_interface name="velocity"/> -->
-            <!-- <state_interface name="effort"/> -->
-        </joint>
-        <joint name="camera_tilt_joint">
-            <command_interface name="position">
-                <param name="min">-3.14</param>
-                <param name="max">3.14</param>
-            </command_interface>
-            <state_interface name="position">
-                <param name="initial_value">0</param>
-            </state_interface>
-            <!-- <state_interface name="velocity"/> -->
-            <!-- <state_interface name="effort"/> -->
-        </joint>
-    </ros2_control>
+    <xacro:unless value="$(arg sim_mode)">
+        <!-- <ros2_control name="RealRobot" type="system">
+            <hardware>
+                <plugin>diffdrive_rpi/DiffDriveRpi</plugin>
+                <param name="left_wheel_name">left_wheel_joint</param>
+                <param name="right_wheel_name">right_wheel_joint</param>
+                <param name="loop_rate">30</param>
+                <param name="device">/dev/ttyUSB0</param>
+                <param name="baud_rate">115200</param>
+                <param name="timeout">1000</param>
+                <param name="enc_counts_per_rev">350</param>
+                <param name="wheel_radius">0.03</param>
+            </hardware>
+            <joint name="left_wheel">
+                <command_interface name="velocity">
+                    <param name="min">-10</param>
+                    <param name="max">10</param>
+                </command_interface>
+                <state_interface name="velocity"/>
+                <state_interface name="position"/>
+            </joint>
+            <joint name="right_wheel">
+                <command_interface name="velocity">
+                    <param name="min">-10</param>
+                    <param name="max">10</param>
+                </command_interface>
+                <state_interface name="velocity"/>
+                <state_interface name="position"/>
+            </joint>
+        </ros2_control> -->
+    </xacro:unless>
+    <xacro:if value="$(arg sim_mode)">
+        <ros2_control name="GazeboSystem" type="system">
+            <hardware>
+                <plugin>gazebo_ros2_control/GazeboSystem</plugin>
+            </hardware>
+            <joint name="left_wheel">
+                <command_interface name="velocity">
+                    <param name="min">-10</param>
+                    <param name="max">10</param>
+                </command_interface>
+                <state_interface name="velocity"/>
+                <state_interface name="position"/>
+            </joint>
+            <joint name="right_wheel">
+                <command_interface name="velocity">
+                    <param name="min">-10</param>
+                    <param name="max">10</param>
+                </command_interface>
+                <state_interface name="velocity"/>
+                <state_interface name="position"/>
+            </joint>
+            <joint name="camera_pan_joint">
+                <command_interface name="position">
+                    <param name="min">-3.14</param>
+                    <param name="max">3.14</param>
+                </command_interface>
+                <state_interface name="position">
+                    <param name="initial_value">0</param>
+                </state_interface>
+                <!-- <state_interface name="velocity"/> -->
+                <!-- <state_interface name="effort"/> -->
+            </joint>
+            <joint name="camera_tilt_joint">
+                <command_interface name="position">
+                    <param name="min">-3.14</param>
+                    <param name="max">3.14</param>
+                </command_interface>
+                <state_interface name="position">
+                    <param name="initial_value">0</param>
+                </state_interface>
+                <!-- <state_interface name="velocity"/> -->
+                <!-- <state_interface name="effort"/> -->
+            </joint>
+        </ros2_control>
+    </xacro:if>
     <gazebo>
         <plugin name="gazebo_ros2_control" filename="libgazebo_ros2_control.so">
